File: schematic.sch (EAGLE design)
At the start: 32 parts, among them Q3 IRF540

Commit message: Add new board
Parts:
- Q1: value (none) -> FDN360P; device transistor-power:PMOSFET_PTO220BV -> transistor-power:FDN360P
- Q3: value IRF540 -> BSS123; device transistor-power:IRF540 -> transistor-small-signal:BSS123
Changed lines of the file:
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@@
 <parts>
 <part name="U$1" library="ic-ds2715-nimh-charger" deviceset="DS2715" device=""/>
-<part name="Q3" library="transistor-power" library_urn="urn:adsk.eagle:library:400" deviceset="IRF540" device=""/>
 <part name="LOAD" library="SparkFun-Connectors" deviceset="CONN_02" device="POLAR"/>
 <part name="POWER" library="SparkFun-Connectors" deviceset="CONN_02" device="POLAR"/>
@@
 <part name="C5" library="rcl" library_urn="urn:adsk.eagle:library:334" deviceset="C-EU" device="025-025X050" value="1nF"/>
 <part name="R5" library="rcl" library_urn="urn:adsk.eagle:library:334" deviceset="R-EU_" device="0207/10" value="160k"/>
-<part name="Q1" library="transistor-power" library_urn="urn:adsk.eagle:library:400" deviceset="PMOSFET_P" device="TO220BV"/>
 <part name="D1" library="diode" library_urn="urn:adsk.eagle:library:210" deviceset="1N581*" device="" technology="7-B"/>
 <part name="D5" library="diode" library_urn="urn:adsk.eagle:library:210" deviceset="1N581*" device="" technology="7-B"/>
 <part name="Q5" library="transistor-power" library_urn="urn:adsk.eagle:library:400" deviceset="PMOSFET_P" device="TO220BV"/>
+<part name="Q1" library="transistor-power" library_urn="urn:adsk.eagle:library:400" deviceset="FDN360P" device=""/>
+<part name="Q3" library="transistor-small-signal" library_urn="urn:adsk.eagle:library:401" deviceset="BSS123" device=""/>
 </parts>
 <sheets>
@@
 <instances>
 <instance part="U$1" gate="G$1" x="35.56" y="68.58"/>
-<instance part="Q3" gate="G$1" x="20.32" y="109.22"/>
 <instance part="LOAD" gate="G$1" x="-15.24" y="139.7" rot="R270"/>
 <instance part="POWER" gate="G$1" x="-66.04" y="106.68"/>
@@
 <instance part="C5" gate="G$1" x="5.08" y="96.52"/>
 <instance part="R5" gate="G$1" x="10.16" y="76.2"/>
-<instance part="Q1" gate="G$1" x="53.34" y="111.76" rot="R90"/>
 <instance part="D1" gate="G$1" x="-35.56" y="109.22"/>
 <instance part="D5" gate="G$1" x="63.5" y="106.68" rot="R90"/>
 <instance part="Q5" gate="G$1" x="2.54" y="127" rot="R90"/>
+<instance part="Q1" gate="G$1" x="53.34" y="111.76" rot="R90"/>
+<instance part="Q3" gate="G$1" x="22.86" y="109.22"/>
 </instances>
 <busses>
@@
 <wire x1="63.5" y1="109.22" x2="63.5" y2="114.3" width="0.1524" layer="91"/>
 <junction x="63.5" y="114.3"/>
+<pinref part="D5" gate="G$1" pin="C"/>
 <pinref part="Q1" gate="G$1" pin="D"/>
-<pinref part="D5" gate="G$1" pin="C"/>
 </segment>
 </net>
@@
 <pinref part="R3" gate="G$1" pin="2"/>
 <wire x1="20.32" y1="101.6" x2="22.86" y2="101.6" width="0.1524" layer="91"/>
-<pinref part="Q3" gate="G$1" pin="S"/>
 <wire x1="22.86" y1="101.6" x2="40.64" y2="101.6" width="0.1524" layer="91"/>
 <wire x1="22.86" y1="104.14" x2="22.86" y2="101.6" width="0.1524" layer="91"/>
 <junction x="22.86" y="101.6"/>
+<wire x1="50.8" y1="101.6" x2="40.64" y2="101.6" width="0.1524" layer="91"/>
 <pinref part="Q1" gate="G$1" pin="G"/>
-<wire x1="50.8" y1="106.68" x2="50.8" y2="101.6" width="0.1524" layer="91"/>
-<wire x1="50.8" y1="101.6" x2="40.64" y2="101.6" width="0.1524" layer="91"/>
+<wire x1="50.8" y1="109.22" x2="50.8" y2="101.6" width="0.1524" layer="91"/>
+<pinref part="Q3" gate="G$1" pin="S"/>
 </segment>
 </net>
@@
 <segment>
 <wire x1="5.08" y1="99.06" x2="5.08" y2="101.6" width="0.1524" layer="91"/>
-<pinref part="Q3" gate="G$1" pin="G"/>
 <wire x1="5.08" y1="101.6" x2="5.08" y2="106.68" width="0.1524" layer="91"/>
 <wire x1="5.08" y1="106.68" x2="17.78" y2="106.68" width="0.1524" layer="91"/>
@@
 <wire x1="10.16" y1="101.6" x2="5.08" y2="101.6" width="0.1524" layer="91"/>
 <junction x="5.08" y="101.6"/>
+<pinref part="Q3" gate="G$1" pin="G"/>
 </segment>
 </net>
@@
 <pinref part="R6" gate="G$1" pin="2"/>
 <wire x1="40.64" y1="114.3" x2="48.26" y2="114.3" width="0.1524" layer="91"/>
-<pinref part="Q3" gate="G$1" pin="D"/>
 <wire x1="40.64" y1="114.3" x2="22.86" y2="114.3" width="0.1524" layer="91"/>
 <junction x="40.64" y="114.3"/>
 <wire x1="22.86" y1="114.3" x2="17.78" y2="114.3" width="0.1524" layer="91"/>
-<junction x="22.86" y="114.3"/>
 <wire x1="17.78" y1="114.3" x2="-5.08" y2="114.3" width="0.1524" layer="91"/>
 <wire x1="-5.08" y1="114.3" x2="-5.08" y2="109.22" width="0.1524" layer="91"/>
@@
 <junction x="-30.48" y="78.74"/>
 <junction x="-25.4" y="109.22"/>
-<pinref part="Q1" gate="G$1" pin="S"/>
 <pinref part="D1" gate="G$1" pin="C"/>
 <pinref part="Q5" gate="G$1" pin="S"/>
-</segment>
-</net>
+<pinref part="Q1" gate="G$1" pin="S"/>
+<pinref part="Q3" gate="G$1" pin="D"/>
+<junction x="22.86" y="114.3"/>
+</segment>
+</net>
