File: schematic_old.brd (EAGLE design)
At the start: 57.1 x 54.6 mm, 32 parts, among them Q3 IRF540

Commit message: Add new board
Parts:
- Q1: value (none) -> FDN360P; device transistor-power:TO220BV -> transistor-power:SUPER-SOT3
- Q3: value IRF540 -> BSS123; device transistor-power:TO220BV -> transistor-small-signal:SOT23
- moved Q3 2.75 mm to (21.6, 46.7)
- moved Q1 2.50 mm to (50.3, 27.7)
Connections:
- net N$10: now also Q1.3; no longer Q1.D
- net N$13: now also Q1.1, Q3.2; no longer Q1.G, Q3.S
- net N$14: now also Q3.1; no longer Q3.G
- net N$26: now also Q1.2, Q3.3; no longer Q1.S, Q3.D
Routing:
- net N$14: track 16.3 -> 12.3 mm
- net N$13: track 59.2 -> 61.9 mm
- net N$26: track 116.5 -> 117.7 mm
- net N$10: track 11.6 -> 12.3 mm
Changed lines of the file:
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@@
 <attribute name="SF_ID" value="PRT-09918" x="62.484" y="26.416" size="1.778" layer="27" rot="R90" display="off"/>
 </element>
-<element name="Q3" library="transistor-power" library_urn="urn:adsk.eagle:library:400" package="TO220BV" value="IRF540" x="23.876" y="48.26" rot="R270"/>
 <element name="R1" library="rcl" library_urn="urn:adsk.eagle:library:334" package="0207/10" value="150" x="56.896" y="43.18" rot="R270"/>
 <element name="R10" library="rcl" library_urn="urn:adsk.eagle:library:334" package="0207/10" value="10k" x="62.992" y="46.736" rot="R270"/>
@@
 <element name="THM" library="SparkFun-Connectors" package="1X02" value="" x="43.18" y="54.864"/>
 <element name="U$1" library="ic-ds2715-nimh-charger" package="DS2715-SO16" value="DS2715" x="43.434" y="47.498"/>
-<element name="Q1" library="transistor-power" library_urn="urn:adsk.eagle:library:400" package="TO220BV" value="" x="52.578" y="28.702" rot="R270"/>
 <element name="D1" library="diode" library_urn="urn:adsk.eagle:library:210" package="DO41-7.6" value="1N5817-B" x="24.13" y="22.352" rot="R90"/>
 <element name="D5" library="diode" library_urn="urn:adsk.eagle:library:210" package="DO41-7.6" value="1N5817-B" x="46.228" y="23.114" rot="R270"/>
 <element name="Q5" library="transistor-power" library_urn="urn:adsk.eagle:library:400" package="TO220BV" value="" x="21.59" y="21.082" rot="R270"/>
+<element name="Q1" library="transistor-power" library_urn="urn:adsk.eagle:library:400" package="SUPER-SOT3" value="FDN360P" x="50.292" y="27.686" rot="R270"/>
+<element name="Q3" library="transistor-small-signal" library_urn="urn:adsk.eagle:library:401" package="SOT23" value="BSS123" x="21.59" y="46.736" rot="R270"/>
 </elements>
 <signals>
@@
 <signal name="N$10">
 <contactref element="L1" pad="1"/>
-<contactref element="Q1" pad="D"/>
 <contactref element="D5" pad="C"/>
-<wire x1="46.228" y1="28.067" x2="46.228" y2="26.924" width="0.5588" layer="1"/>
+<wire x1="46.228" y1="27.686" x2="46.228" y2="28.067" width="0.5588" layer="1"/>
+<wire x1="46.228" y1="27.686" x2="46.228" y2="26.924" width="0.5588" layer="1"/>
 <wire x1="46.228" y1="28.067" x2="45.593" y2="28.702" width="0.5588" layer="1"/>
-<wire x1="46.228" y1="26.924" x2="46.228" y2="29.464" width="1.778" layer="1"/>
+<wire x1="46.228" y1="26.924" x2="46.228" y2="27.686" width="1.778" layer="1"/>
+<wire x1="46.228" y1="27.686" x2="46.228" y2="29.464" width="1.778" layer="1"/>
 <wire x1="46.228" y1="29.464" x2="44.831" y2="29.464" width="1.778" layer="1"/>
 <wire x1="44.704" y1="29.464" x2="44.831" y2="29.464" width="1.778" layer="1"/>
-<wire x1="50.038" y1="28.702" x2="45.593" y2="28.702" width="1.778" layer="1"/>
 <wire x1="45.593" y1="28.702" x2="44.831" y2="29.464" width="1.778" layer="1"/>
+<contactref element="Q1" pad="3"/>
+<wire x1="51.392" y1="27.686" x2="46.228" y2="27.686" width="0.1524" layer="1"/>
 </signal>
 <signal name="N$12">
@@
 <contactref element="R9" pad="2"/>
 <contactref element="R3" pad="2"/>
-<contactref element="Q3" pad="S"/>
-<contactref element="Q1" pad="G"/>
 <via x="49.276" y="37.846" extent="1-16" drill="0.9"/>
 <wire x1="49.276" y1="37.846" x2="34.29" y2="37.846" width="0.5588" layer="16"/>
 <via x="34.29" y="37.846" extent="1-16" drill="0.9"/>
-<wire x1="49.276" y1="37.846" x2="49.276" y2="31.242" width="1.016" layer="1"/>
-<wire x1="49.276" y1="31.242" x2="50.038" y2="31.242" width="1.016" layer="1"/>
+<wire x1="49.276" y1="31.242" x2="49.276" y2="37.846" width="1.016" layer="1"/>
 <wire x1="34.29" y1="37.846" x2="34.29" y2="40.64" width="1.016" layer="1"/>
 <wire x1="34.29" y1="40.64" x2="26.416" y2="40.64" width="1.016" layer="1"/>
@@
 <wire x1="26.416" y1="36.068" x2="30.48" y2="36.068" width="1.016" layer="1"/>
 <wire x1="30.48" y1="36.068" x2="30.48" y2="28.702" width="1.016" layer="1"/>
-<wire x1="26.416" y1="40.64" x2="26.416" y2="45.72" width="1.016" layer="1"/>
-<wire x1="26.416" y1="45.72" x2="21.336" y2="45.72" width="1.016" layer="1"/>
+<wire x1="26.416" y1="45.72" x2="26.416" y2="40.64" width="1.016" layer="1"/>
+<contactref element="Q1" pad="1"/>
+<contactref element="Q3" pad="2"/>
+<wire x1="49.192" y1="28.636" x2="49.192" y2="31.158" width="0.1524" layer="1"/>
+<wire x1="49.192" y1="31.158" x2="49.276" y2="31.242" width="0.1524" layer="1"/>
+<wire x1="20.49" y1="45.786" x2="26.35" y2="45.786" width="0.1524" layer="1"/>
+<wire x1="26.35" y1="45.786" x2="26.416" y2="45.72" width="0.1524" layer="1"/>
 </signal>
 <signal name="N$14">
-<contactref element="Q3" pad="G"/>
 <contactref element="C5" pad="1"/>
 <contactref element="R3" pad="1"/>
-<wire x1="26.416" y1="50.8" x2="21.336" y2="50.8" width="0.5588" layer="1"/>
-<wire x1="29.464" y1="50.8" x2="26.416" y2="50.8" width="0.5588" layer="1"/>
-<wire x1="21.336" y1="50.8" x2="29.464" y2="50.8" width="1.016" layer="1"/>
+<wire x1="26.416" y1="50.8" x2="29.464" y2="50.8" width="0.5588" layer="1"/>
+<contactref element="Q3" pad="1"/>
+<wire x1="20.49" y1="47.686" x2="20.49" y2="50.63" width="0.1524" layer="1"/>
+<wire x1="20.49" y1="50.63" x2="20.32" y2="50.8" width="0.1524" layer="1"/>
+<wire x1="20.32" y1="50.8" x2="26.416" y2="50.8" width="0.1524" layer="1"/>
 </signal>
 <signal name="N$9">
@@
 <contactref element="C2" pad="1"/>
 <contactref element="R6" pad="2"/>
-<contactref element="Q3" pad="D"/>
 <contactref element="LOAD" pad="2"/>
 <contactref element="LED1" pad="A"/>
 <contactref element="D2" pad="A"/>
 <contactref element="D4" pad="C"/>
-<contactref element="Q1" pad="S"/>
 <contactref element="D1" pad="C"/>
 <contactref element="Q5" pad="S"/>
@@
 <wire x1="37.084" y1="18.542" x2="39.116" y2="18.542" width="1.27" layer="1"/>
 <wire x1="39.624" y1="24.384" x2="41.656" y2="24.384" width="1.27" layer="1"/>
-<wire x1="21.336" y1="48.26" x2="16.002" y2="48.26" width="1.778" layer="1"/>
-<wire x1="16.002" y1="48.26" x2="16.002" y2="37.084" width="1.778" layer="1"/>
+<wire x1="16.002" y1="46.736" x2="16.002" y2="48.26" width="1.778" layer="1"/>
+<wire x1="16.002" y1="46.736" x2="16.002" y2="37.084" width="1.778" layer="1"/>
 <wire x1="16.002" y1="37.084" x2="19.304" y2="37.084" width="1.778" layer="1"/>
 <wire x1="16.002" y1="37.084" x2="16.002" y2="33.274" width="1.778" layer="1"/>
@@
 <wire x1="39.116" y1="24.384" x2="41.656" y2="24.384" width="1.778" layer="1"/>
 <wire x1="41.656" y1="24.384" x2="44.958" y2="24.384" width="1.778" layer="1"/>
-<wire x1="44.958" y1="24.384" x2="50.038" y2="20.32" width="1.778" layer="1"/>
-<wire x1="50.038" y1="20.32" x2="50.038" y2="26.162" width="1.778" layer="1"/>
+<wire x1="48.953853125" y1="21.187315625" x2="44.958" y2="24.384" width="1.778" layer="1"/>
+<contactref element="Q1" pad="2"/>
+<contactref element="Q3" pad="3"/>
+<wire x1="48.953853125" y1="21.187315625" x2="50.038" y2="20.32" width="1.778" layer="1"/>
+<wire x1="49.192" y1="26.736" x2="49.192" y2="21.4254625" width="0.1524" layer="1"/>
+<wire x1="49.192" y1="21.4254625" x2="48.953853125" y2="21.187315625" width="0.1524" layer="1"/>
+<wire x1="22.69" y1="46.736" x2="16.002" y2="46.736" width="0.1524" layer="1"/>
 </signal>
 <signal name="N$1">
